File: huibike.kicad_sch (KiCad schematic)
At the start: 17 parts, among them J101 Sensor, Q101 BC847, U101 ATtiny10-TS, U102 LM78M05_TO252

Commit message: Update Parts
Parts:
- C101, C103: DistribPart# (none) -> C28323; Distributor (none) -> JLPCB; ManuPart# (none) -> CL21B105KBFNNNE; Manufacture (none) -> Samsung Electro-Mechanics; assemble (none) -> y
- C102, C104: DistribPart# (none) -> C1525; Distributor (none) -> JLPCB; ManuPart# (none) -> CL05B104KO5NNNC; Manufacture (none) -> Samsung Electro-Mechanics; assemble (none) -> y
- D101, D102: DistribPart# (none) -> C8056; Distributor (none) -> JLPCB; ManuPart# (none) -> ZMM3V3-M; Manufacture (none) -> ST(Semtech); assemble (none) -> y
- J101, JP101: DistribPart# (none) -> N/A; Distributor (none) -> N/A; ManuPart# (none) -> N/A; Manufacture (none) -> N/A; assemble (none) -> n
- Q101: DistribPart# (none) -> C475630; Distributor (none) -> JLPCB; ManuPart# (none) -> BC847; Manufacture (none) -> Shikues; assemble (none) -> y
- R101, R102, R103, R104, R105, R106: DistribPart# (none) -> C25756; Distributor (none) -> JLPCB; ManuPart# (none) -> 0402WGF1502TCE; Manufacture (none) -> UNI-ROYAL(Uniroyal Elec); assemble (none) -> y
- U101: DistribPart# (none) -> C128438; Distributor (none) -> JLPCB; ManuPart# (none) -> ATTINY10-TSHR; Manufacture (none) -> Microchip Tech; assemble (none) -> y
- U102: DistribPart# (none) -> C58069; Distributor (none) -> JLPCB; ManuPart# (none) -> L78M05ABDT-TR; Manufacture (none) -> STMicroelectronics; assemble (none) -> y
